Commit message: fix(description): 激光雷达旋转改为 0 度

File: src/rm_ep_description/urdf/sensor.urdf.xacro (robot description, xacro)
@@ -5,5 +5,5 @@
     <link name="${tf_prefix}laser_link"/>
     <joint name="${tf_prefix}base_to_laser" type="fixed">
-      <origin xyz="0 0 0.15" rpy="0 0 ${pi}"/>
+      <origin xyz="0 0 0.15" rpy="0 0 0"/>
       <parent link="${tf_prefix}base_link"/>
       <child link="${tf_prefix}laser_link"/>
